File: KiCad/MSK_RF.kicad_sch (KiCad schematic)
At the start: 65 parts, among them J1 Conn_01x05_Male, J2 Conn_01x12, J3 Conn_01x12, J4 Conn_Coaxial, J5 47346-0001, U1 STM32WLE5CCU6, U2 ADG918BRM, U3 TLV70233_SOT23-5, Y1 32.768 kHz, Y2 ECS-320-8-37-CKM-TR3

Commit message: documentation and description
Other:
- note added: "SWD connector"
- note added: "Voltage divider"
- note removed: "SWD conn"
- note removed: "Używamy SWD więc BOOT0 do GND"
- note removed: "VDD dla switcha to 2.75V, sam switch bierze <1uA to dałem zwykły dzielnik napięcia z 3.3V na 2.75V"
- note removed: "W datasheet zalecają serie X5R/X7R ceramicznych capów wartość capa na wyjściu >=1uF"
- moved on the sheet: J1
Changed lines of the file:
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@@
+    (stroke (width 0) (type default) (color 0 0 0 0))
+  )
+  (polyline (pts (xy 135.89 110.49) (xy 135.89 130.81))
     (stroke (width 0) (type default) (color 0 0 0 0))
   )
@@
     (stroke (width 0) (type default) (color 0 0 0 0))
   )
+  (polyline (pts (xy 179.07 105.41) (xy 135.89 105.41))
+    (stroke (width 0) (type default) (color 0 0 0 0))
+  )
   (wire (pts (xy 62.23 133.35) (xy 62.23 135.89))
     (stroke (width 0) (type default) (color 0 0 0 0))
@@
     (stroke (width 0) (type default) (color 0 0 0 0))
   )
+  (polyline (pts (xy 135.89 130.81) (xy 179.07 130.81))
+    (stroke (width 0) (type default) (color 0 0 0 0))
+  )
   (wire (pts (xy 163.83 50.8) (xy 177.8 50.8))
     (stroke (width 0) (type default) (color 0 0 0 0))
   )
+  (polyline (pts (xy 135.89 105.41) (xy 135.89 110.49))
+    (stroke (width 0) (type default) (color 0 0 0 0))
+  )
   (wire (pts (xy 87.63 133.35) (xy 93.98 133.35))
     (stroke (width 0) (type default) (color 0 0 0 0))
@@
     (stroke (width 0) (type default) (color 0 0 0 0))
   )
-  (wire (pts (xy 149.86 102.87) (xy 163.83 102.87))
+  (wire (pts (xy 153.67 121.92) (xy 167.64 121.92))
     (stroke (width 0) (type default) (color 0 0 0 0))
   )
@@
     (stroke (width 0) (type default) (color 0 0 0 0))
   )
-  (wire (pts (xy 163.83 97.79) (xy 149.86 97.79))
+  (wire (pts (xy 167.64 116.84) (xy 153.67 116.84))
     (stroke (width 0) (type default) (color 0 0 0 0))
   )
@@
     (stroke (width 0) (type default) (color 0 0 0 0))
   )
+  (polyline (pts (xy 179.07 130.81) (xy 179.07 105.41))
+    (stroke (width 0) (type default) (color 0 0 0 0))
+  )
   (wire (pts (xy 33.02 54.61) (xy 45.72 54.61))
     (stroke (width 0) (type default) (color 0 0 0 0))
@@
     (stroke (width 0) (type default) (color 0 0 0 0))
   )
-  (wire (pts (xy 149.86 95.25) (xy 163.83 95.25))
+  (wire (pts (xy 153.67 114.3) (xy 167.64 114.3))
     (stroke (width 0) (type default) (color 0 0 0 0))
   )
@@
     (stroke (width 0) (type default) (color 0 0 0 0))
   )
-  (wire (pts (xy 163.83 100.33) (xy 149.86 100.33))
+  (wire (pts (xy 167.64 119.38) (xy 153.67 119.38))
     (stroke (width 0) (type default) (color 0 0 0 0))
   )
@@
     (stroke (width 0) (type default) (color 0 0 0 0))
   )
-  (wire (pts (xy 149.86 105.41) (xy 163.83 105.41))
+  (wire (pts (xy 153.67 124.46) (xy 167.64 124.46))
     (stroke (width 0) (type default) (color 0 0 0 0))
   )
@@
     (stroke (width 0) (type default) (color 0 0 0 0))
   )
-  (text "W datasheet zalecają serie X5R/X7R ceramicznych capów\nwartość capa na wyjściu >=1uF"
-    (at 238.76 110.49 0)
-    (effects (font (size 1.27 1.27)) (justify left bottom))
-  )
-  (text "Używamy SWD więc BOOT0 do GND" (at 270.51 80.01 0)
-    (effects (font (size 1.27 1.27)) (justify left bottom))
-  )
-  (text "SWD conn" (at 151.13 90.17 0)
+  (text "SWD connector" (at 152.4 104.14 0)
     (effects (font (size 1.27 1.27)) (justify left bottom))
   )
@@
     (effects (font (size 1.27 1.27)) (justify left bottom))
   )
-  (text "VDD dla switcha to 2.75V, sam switch bierze <1uA\nto dałem zwykły dzielnik napięcia z 3.3V na 2.75V"
-    (at 229.87 368.3 0)
+  (text "Voltage divider" (at 246.38 365.76 0)
     (effects (font (size 1.27 1.27)) (justify left bottom))
   )
@@
     (effects (font (size 1.27 1.27)) (justify left bottom))
   )
-  (label "SWCLK" (at 162.56 100.33 180)
+  (label "SWCLK" (at 166.37 119.38 180)
     (effects (font (size 1.27 1.27)) (justify right bottom))
   )
@@
     (effects (font (size 1.27 1.27)) (justify left bottom))
   )
-  (label "SWDIO" (at 162.56 97.79 180)
+  (label "SWDIO" (at 166.37 116.84 180)
     (effects (font (size 1.27 1.27)) (justify right bottom))
   )
@@
     )
   )
-  (global_label "PA13" (shape bidirectional) (at 163.83 97.79 0) (fields_autoplaced)
-    (effects (font (size 1.27 1.27)) (justify left))
-    (property "Intersheet References" "${INTERSHEET_REFS}" (id 0) (at 171.0207 97.7106 0)
-      (effects (font (size 1.27 1.27)) (justify left) hide)
-    )
-  )
-  (global_label "PA14" (shape bidirectional) (at 163.83 100.33 0) (fields_autoplaced)
-    (effects (font (size 1.27 1.27)) (justify left))
-    (property "Intersheet References" "${INTERSHEET_REFS}" (id 0) (at 171.0207 100.4094 0)
-      (effects (font (size 1.27 1.27)) (justify left) hide)
-    )
-  )
-  (global_label "GND" (shape bidirectional) (at 163.83 105.41 0) (fields_autoplaced)
-    (effects (font (size 1.27 1.27)) (justify left))
-    (property "Intersheet References" "${INTERSHEET_REFS}" (id 0) (at 170.1136 105.4894 0)
+  (global_label "PA13" (shape bidirectional) (at 167.64 116.84 0) (fields_autoplaced)
+    (effects (font (size 1.27 1.27)) (justify left))
+    (property "Intersheet References" "${INTERSHEET_REFS}" (id 0) (at 174.8307 116.7606 0)
+      (effects (font (size 1.27 1.27)) (justify left) hide)
+    )
+  )
+  (global_label "PA14" (shape bidirectional) (at 167.64 119.38 0) (fields_autoplaced)
+    (effects (font (size 1.27 1.27)) (justify left))
+    (property "Intersheet References" "${INTERSHEET_REFS}" (id 0) (at 174.8307 119.4594 0)
+      (effects (font (size 1.27 1.27)) (justify left) hide)
+    )
+  )
+  (global_label "GND" (shape bidirectional) (at 167.64 124.46 0) (fields_autoplaced)
+    (effects (font (size 1.27 1.27)) (justify left))
+    (property "Intersheet References" "${INTERSHEET_REFS}" (id 0) (at 173.9236 124.5394 0)
       (effects (font (size 1.27 1.27)) (justify left) hide)
     )
@@
     )
   )
-  (global_label "NRST" (shape bidirectional) (at 163.83 102.87 0) (fields_autoplaced)
-    (effects (font (size 1.27 1.27)) (justify left))
-    (property "Intersheet References" "${INTERSHEET_REFS}" (id 0) (at 171.0207 102.7906 0)
+  (global_label "NRST" (shape bidirectional) (at 167.64 121.92 0) (fields_autoplaced)
+    (effects (font (size 1.27 1.27)) (justify left))
+    (property "Intersheet References" "${INTERSHEET_REFS}" (id 0) (at 174.8307 121.8406 0)
       (effects (font (size 1.27 1.27)) (justify left) hide)
     )
@@
     )
   )
-  (global_label "3.3V" (shape bidirectional) (at 163.83 95.25 0) (fields_autoplaced)
-    (effects (font (size 1.27 1.27)) (justify left))
-    (property "Intersheet References" "${INTERSHEET_REFS}" (id 0) (at 170.3555 95.1706 0)
+  (global_label "3.3V" (shape bidirectional) (at 167.64 114.3 0) (fields_autoplaced)
+    (effects (font (size 1.27 1.27)) (justify left))
+    (property "Intersheet References" "${INTERSHEET_REFS}" (id 0) (at 174.1655 114.2206 0)
       (effects (font (size 1.27 1.27)) (justify left) hide)
     )
@@
     (pin "1")
   )
-  (symbol (lib_id "Connector:Conn_01x05_Male") (at 144.78 100.33 0) (unit 1)
-    (in_bom yes) (on_board yes) (fields_autoplaced)
-    (property "Reference" "J1" (id 0) (at 145.415 90.17 0))
-    (property "Value" "Conn_01x05_Male" (id 1) (at 145.415 92.71 0))
-    (property "Footprint" "Connector_PinHeader_2.54mm:PinHeader_1x05_P2.54mm_Vertical" (id 2) (at 144.78 100.33 0)
-      (effects (font (size 1.27 1.27)) hide)
-    )
-    (property "Datasheet" "~" (id 3) (at 144.78 100.33 0)
-      (effects (font (size 1.27 1.27)) hide)
-    )
+  (symbol (lib_id "Connector:Conn_01x05_Male") (at 148.59 119.38 0) (unit 1)
+    (in_bom yes) (on_board yes) (fields_autoplaced)
+    (property "Reference" "J1" (id 0) (at 149.225 109.22 0))
+    (property "Value" "Conn_01x05_Male" (id 1) (at 149.225 111.76 0))
+    (property "Footprint" "Connector_PinHeader_2.54mm:PinHeader_1x05_P2.54mm_Vertical" (id 2) (at 148.59 119.38 0)
+      (effects (font (size 1.27 1.27)) hide)
+    )
+    (property "Datasheet" "~" (id 3) (at 148.59 119.38 0)
+      (effects (font (size 1.27 1.27)) hide)
+    )
